Commit message: Feature : cmd_vel joint control

File: sw_ros2_control_gazebo/urdf/vel_model.urdf (robot description, URDF)
Before this commit: robot rotate_box_bot, 4 links, 3 joints
Joints:
- joint link_1_JOINT_0: limit lower=-1.22173 upper=1.22173 effort=1000.0 velocity=0.1 -> effort=10 velocity=100; type revolute -> continuous
