Commit message: Fix : revolute joint limit

File: sw_ros2_control_gazebo/urdf/position_forward_model.urdf (robot description, URDF)
Before this commit: robot rotate_box_bot, 4 links, 3 joints
Joints:
- joint link_1_JOINT_0: limit lower=-1.22173 upper=1.22173 effort=1000.0 velocity=0.1 -> lower=-3.1415 upper=3.1415 effort=1000.0 velocity=0.1

File: sw_ros2_control_gazebo/urdf/position_traj_model.urdf (robot description, URDF)
Before this commit: robot rotate_box_bot, 4 links, 3 joints
Joints:
- joint link_1_JOINT_0: limit lower=-1.22173 upper=1.22173 effort=1000.0 velocity=0.1 -> lower=-3.1415 upper=3.1415 effort=1000.0 velocity=0.1

Commit message: Fix : unmatched joint position

File: sw_ros2_control_gazebo/urdf/position_forward_model.urdf (robot description, URDF)
Before this commit: robot rotate_box_bot, 4 links, 3 joints
Joints:
- joint link_0_JOINT_0: origin xyz=0 0 1 rpy=0 0 0 -> xyz=0 0 0 rpy=0 0 0

File: sw_ros2_control_gazebo/urdf/position_traj_model.urdf (robot description, URDF)
Before this commit: robot rotate_box_bot, 4 links, 3 joints
Joints:
- joint link_0_JOINT_0: origin xyz=0 0 1 rpy=0 0 0 -> xyz=0 0 0 rpy=0 0 0

File: sw_ros2_control_gazebo/urdf/vel_model.urdf (robot description, URDF)
Before this commit: robot rotate_box_bot, 4 links, 3 joints
Joints:
- joint link_0_JOINT_0: origin xyz=0 0 1 rpy=0 0 0 -> xyz=0 0 0 rpy=0 0 0
