Commit message: Feature : racecar simulation

File: sw_ros2_control_gazebo/urdf/racecar/macros.xacro (robot description, xacro)
@@ -41,5 +41,5 @@
   <origin xyz="0 0 0" rpy="0 0 0" />
   <geometry>
-    <mesh filename="$(find diffbot_description)/meshes/chassis.STL" />
+    <mesh filename="$(find sw_ros2_control_gazebo)/meshes/chassis.STL" />
   </geometry>
 </xacro:macro>
@@ -47,5 +47,5 @@
   <origin xyz="0 0 0" rpy="0 0 0" />
   <geometry>
-    <mesh filename="$(find diffbot_description)/meshes/left_rear_wheel.STL" />
+    <mesh filename="$(find sw_ros2_control_gazebo)/meshes/left_rear_wheel.STL" />
   </geometry>
 </xacro:macro>
@@ -53,5 +53,5 @@
   <origin xyz="0 0 0" rpy="0 0 0" />
   <geometry>
-    <mesh filename="$(find diffbot_description)/meshes/right_rear_wheel.STL" />
+    <mesh filename="$(find sw_ros2_control_gazebo)/meshes/right_rear_wheel.STL" />
   </geometry>
 </xacro:macro>
@@ -59,5 +59,5 @@
   <origin xyz="0 0 0" rpy="0 0 0" />
   <geometry>
-    <mesh filename="$(find diffbot_description)/meshes/left_front_wheel.STL" />
+    <mesh filename="$(find sw_ros2_control_gazebo)/meshes/left_front_wheel.STL" />
   </geometry>
 </xacro:macro>
@@ -65,5 +65,5 @@
   <origin xyz="0 0 0" rpy="0 0 0" />
   <geometry>
-    <mesh filename="$(find diffbot_description)/meshes/right_front_wheel.STL" />
+    <mesh filename="$(find sw_ros2_control_gazebo)/meshes/right_front_wheel.STL" />
   </geometry>
 </xacro:macro>
@@ -71,5 +71,5 @@
   <origin xyz="0 0 0" rpy="0 0 0" />
   <geometry>
-    <mesh filename="$(find diffbot_description)/meshes/left_steering_hinge.STL" />
+    <mesh filename="$(find sw_ros2_control_gazebo)/meshes/left_steering_hinge.STL" />
   </geometry>
 </xacro:macro>
@@ -77,5 +77,5 @@
   <origin xyz="0 0 0" rpy="0 0 0" />
   <geometry>
-    <mesh filename="$(find diffbot_description)/meshes/right_steering_hinge.STL" />
+    <mesh filename="$(find sw_ros2_control_gazebo)/meshes/right_steering_hinge.STL" />
   </geometry>
 </xacro:macro>

File: sw_ros2_control_gazebo/urdf/racecar/racecar.urdf (robot description, URDF)
Before this commit: robot racecar, 13 links, 12 joints
Links:
- link chassis: geometry visual mesh filename=/home/kimsooyoung/ros2_ws/install/sw_ros2_control_gazebo/sh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
- link left_front_wheel: geometry collision cylinder length=0.045 radius=0.05; visual mesh filename=/home/kimsooyoung/ros2_ws/install/sw_ros2_control_gazebo/sh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
- link left_rear_wheel: geometry collision cylinder length=0.045 radius=0.05; visual mesh filename=/home/kimsooyoung/ros2_ws/install/sw_ros2_control_gazebo/sh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
- link left_steering_hinge: geometry visual mesh filename=/home/kimsooyoung/ros2_ws/install/sw_ros2_control_gazebo/sh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
- link right_front_wheel: geometry collision cylinder length=0.045 radius=0.05; visual mesh filename=/home/kimsooyoung/ros2_ws/install/sw_ros2_control_gazebo/sh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
- link right_rear_wheel: geometry collision cylinder length=0.045 radius=0.05; visual mesh filename=/home/kimsooyoung/ros2_ws/install/sw_ros2_control_gazebo/sh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
- link right_steering_hinge: geometry visual mesh filename=/home/kimsooyoung/ros2_ws/install/sw_ros2_control_gazebo/sh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
