Commit message: Feature : gazebo with race course && lidar added

File: sw_ros2_control_gazebo/urdf/racecar/racecar_windows.urdf (robot description, URDF)
Before this commit: robot racecar, 13 links, 12 joints
Links:
- link chassis: geometry visual mesh filename=/home/kimsooyoung/ros2_ws/install/sw_ros2_control_gazebo/sh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
- link laser: geometry collision box size=0.1 0.1 0.1; visual mesh filename=/home/kimsooyoung/ros2_ws/install/sw_ros2_control_gazebo/sh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
- link left_front_wheel: geometry collision cylinder length=0.045 radius=0.05; visual mesh filename=/home/kimsooyoung/ros2_ws/install/sw_ros2_control_gazebo/sh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
- link left_rear_wheel: geometry collision cylinder length=0.045 radius=0.05; visual mesh filename=/home/kimsooyoung/ros2_ws/install/sw_ros2_control_gazebo/sh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
- link left_steering_hinge: geometry visual mesh filename=/home/kimsooyoung/ros2_ws/install/sw_ros2_control_gazebo/sh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
- link right_front_wheel: geometry collision cylinder length=0.045 radius=0.05; visual mesh filename=/home/kimsooyoung/ros2_ws/install/sw_ros2_control_gazebo/sh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
- link right_rear_wheel: geometry collision cylinder length=0.045 radius=0.05; visual mesh filename=/home/kimsooyoung/ros2_ws/install/sw_ros2_control_gazebo/sh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
- link right_steering_hinge: geometry visual mesh filename=/home/kimsooyoung/ros2_ws/install/sw_ros2_control_gazebo/sh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
