Commit message: imu added

File: sw_ros2_control_gazebo/urdf/racecar/racecar.urdf (robot description, URDF)
Before this commit: robot racecar, 13 links, 12 joints
Links:
- added link imu_link, mass 0.01
- link chassis: geometry visual mesh filename=/home/kimsooyoung/ros2_ws/install/sw_ros2_control_gazebo/sh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
- link laser: geometry collision box size=0.1 0.1 0.1; visual mesh filename=/home/kimsooyoung/ros2_ws/install/sw_ros2_control_gazebo/sh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
- link left_front_wheel: geometry collision cylinder length=0.045 radius=0.05; visual mesh filename=/home/kimsooyoung/ros2_ws/install/sw_ros2_control_gazebo/sh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
- link left_rear_wheel: geometry collision cylinder length=0.045 radius=0.05; visual mesh filename=/home/kimsooyoung/ros2_ws/install/sw_ros2_control_gazebo/sh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
- link left_steering_hinge: geometry visual mesh filename=/home/kimsooyoung/ros2_ws/install/sw_ros2_control_gazebo/sh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
- link right_front_wheel: geometry collision cylinder length=0.045 radius=0.05; visual mesh filename=/home/kimsooyoung/ros2_ws/install/sw_ros2_control_gazebo/sh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
- link right_rear_wheel: geometry collision cylinder length=0.045 radius=0.05; visual mesh filename=/home/kimsooyoung/ros2_ws/install/sw_ros2_control_gazebo/sh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
- link right_steering_hinge: geometry visual mesh filename=/home/kimsooyoung/ros2_ws/install/sw_ros2_control_gazebo/sh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
Joints:
- added joint imu_joint: type fixed, parent zed_camera_link, child imu_link, origin xyz=0.01 0 0 rpy=0 0 0

File: sw_ros2_control_gazebo/urdf/racecar/racecar.urdf.xacro (robot description, xacro)
@@ -228,3 +228,15 @@
     <axis xyz="0 0 1" />
   </joint>
+  <link name="imu_link">
+    <inertial>
+      <mass value="0.01"/>
+      <inertia ixx="1.0" ixy="0" ixz="0" iyy="1.0" iyz="0" izz="1.0"/>
+    </inertial>
+  </link>
+  <joint name="imu_joint" type="fixed">
+    <origin xyz="0.01 0 0" rpy="0 0 0"/>
+    <parent link="zed_camera_link"/>
+    <child link="imu_link"/>
+    <!-- <axis xyz="0 0 1" /> -->
+  </joint>
 </robot>

Commit message: Update : params updated

File: sw_ros2_control_gazebo/urdf/racecar/racecar.urdf (robot description, URDF)
Before this commit: robot racecar, 14 links, 13 joints
Joints:
- joint left_steering_hinge_joint: limit lower=-1.0 upper=1.0 effort=10 velocity=100 -> lower=-0.7853 upper=0.7853 effort=10 velocity=100
- joint right_steering_hinge_joint: limit lower=-1.0 upper=1.0 effort=10 velocity=100 -> lower=-0.7853 upper=0.7853 effort=10 velocity=100

File: sw_ros2_control_gazebo/urdf/racecar/racecar.urdf.xacro (robot description, xacro)
@@ -84,5 +84,5 @@
     <child link="left_steering_hinge" />
     <axis xyz="-1 0 0" />
-    <limit lower="-1.0" upper="1.0" effort="10" velocity="100" />
+    <limit lower="-0.7853" upper="0.7853" effort="10" velocity="100" />
   </joint>
   <xacro:steering_hinge_transmission name="left_steering_hinge" />
@@ -102,5 +102,5 @@
     <child link="right_steering_hinge" />
     <axis xyz="-1 0 0" />
-    <limit lower="-1.0" upper="1.0" effort="10" velocity="100" />
+    <limit lower="-0.7853" upper="0.7853" effort="10" velocity="100" />
   </joint>
   <xacro:steering_hinge_transmission name="right_steering_hinge" />
